Commit message: Basically working version of ROS2 porting. Not all parameters are implemented, and some deadlocks occur.
# Conflicts:
#	pf_driver/include/pf_driver/pf/pf_interface.h
#	pf_driver/include/pf_driver/pf/pf_packet.h
#	pf_driver/include/pf_driver/pf/pfsdp_protocol.hpp
#	pf_driver/include/pf_driver/pf/pipeline.h
#	pf_driver/include/pf_driver/pf/r2000/pfsdp_2000.hpp
#	pf_driver/include/pf_driver/pf/r2300/pfsdp_2300.hpp
#	pf_driver/include/pf_driver/ros/scan_publisher.h
#	pf_driver/msg/PFHeader.msg
#	pf_driver/msg/PFR2000Header.msg
#	pf_driver/msg/PFR2300Header.msg
#	pf_driver/src/pf/pf_packet.cpp
#	pf_interfaces/msg/PFHeader.msg
#	pf_interfaces/msg/PFR2000Header.msg
#	pf_interfaces/msg/PFR2300Header.msg
#	src/pf_driver/CMakeLists.txt
#	src/pf_driver/include/pf_driver/pf/pf_parser.h
#	src/pf_driver/msg/PFHeader.msg
#	src/pf_driver/msg/PFR2000Header.msg
#	src/pf_driver/msg/PFR2300Header.msg
#	src/pf_driver/src/pf/pf_interface.cpp
#	src/pf_driver/src/pf/pfsdp_protocol.cpp
#	src/pf_driver/src/ros/pf_data_publisher.cpp
#	src/pf_driver/src/ros/ros_main.cpp
#	src/pf_driver/tests/pfsdp_protocol.cpp

File: src/pf_description/urdf/r2000.urdf.xacro (robot description, xacro)
@@ -4,13 +4,13 @@
         <link name="${prefix}scanner_link" >
             <visual>
-                <origin xyz="0 0 0" rpy="1.57 0 1.57" />
+                <origin xyz="0 0 0" rpy="0 0 0" />
                 <geometry>
-                    <mesh filename="package://pf_description/meshes/R2000.stl" scale="0.001 0.001 0.001" />
+                    <mesh filename="$(find pf_description)/meshes/R2000.dae" />
                 </geometry>
             </visual>
             <collision>
-                <origin xyz="0 0 0.045" rpy="0 0 0" />
+                <origin xyz="-0.0058 0 -0.03885" rpy="0 0 0" />
                 <geometry>
-                    <box size="0.108 0.118 0.128" />
+                    <box size="0.118 0.108 0.117" />
                 </geometry>
             </collision>

File: src/pf_description/urdf/r2300.urdf.xacro (robot description, xacro)
@@ -4,13 +4,13 @@
         <link name="${prefix}scanner_link" >
             <visual>
-                <origin xyz="-0.00195 0.0158 -0.0094" rpy="-1.57 0 1.57" />
+                <origin xyz="0 0 0" rpy="0 0 0" />
                 <geometry>
-                    <mesh filename="package://pf_description/meshes/R2300.stl" scale="0.001 0.001 0.001" />
+                    <mesh filename="$(find pf_description)/meshes/R2300.dae" />
                 </geometry>
             </visual>
             <collision>
-                <origin xyz="-0.00195 0.0158 -0.0094" rpy="-1.57 0 1.57" />
+                <origin xyz="0.01195 0.0158 -0.017" rpy="0 0 0" />
                 <geometry>
-                    <box size="0.0951 0.0685 0.0695" />
+                    <box size="0.07 0.0959 0.0586" />
                 </geometry>
             </collision>
